File: Board/iBaoFeng.sch (EAGLE design)
At the start: 9 parts

Commit message: Changed from audio jacks to headers
Parts:
- removed BAOFENG2.5SPK: (no value), SparkFun-Connectors:AUDIO-JACK2.5MM
- removed BAOFENG3.5MIC: (no value), SparkFun-Connectors:AUDIO-JACKHOLESONLY
- removed IPHONE: AUDIO-JACK3, SparkFun-Connectors:AUDIO-JACK3
- added JP1, JP2: M02PTH3, SparkFun-Connectors:M02PTH3
- added JP3: (no value), SparkFun-Connectors:M04LONGPADS
- D1: device SparkFun-DiscreteSemi:DIODE1N4148 -> SparkFun-DiscreteSemi:DIODESMB
Connections:
- net BAOFENGMIC+: now also JP2.1, JP3.3; no longer BAOFENG3.5MIC.RIGHT, IPHONE.TIP
- net BAOFENGMIC-: now also JP2.2; no longer BAOFENG3.5MIC.SLEEVE
- net BAOFENGSPK+: now also JP1.1; no longer BAOFENG2.5SPK.LEFT
- net GND: now also JP1.2, JP3.1, JP3.4; no longer BAOFENG2.5SPK.SLEEVE, IPHONE.RING2
- net N$4: now also JP3.2; no longer IPHONE.EARTH
